Commit message: 添加realsense仿真

File: models/iris_with_standoffs_new/model.urdf (robot description, URDF)
Before this commit: robot iris, 8 links, 7 joints
Links:
- link base_link: geometry visual cylinder length=0.17 radius=0.005; visual cylinder length=0.17 radius=0.005
- link rotor_0: geometry visual mesh filename=file:///home/hggshiwo/catkin_ws/src/gazebo_sim/models/iris_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 scale=1 1 1
- link rotor_1: geometry visual mesh filename=file:///home/hggshiwo/catkin_ws/src/gazebo_sim/models/iris_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 scale=1 1 1
- link rotor_2: geometry visual mesh filename=file:///home/hggshiwo/catkin_ws/src/gazebo_sim/models/iris_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 scale=1 1 1
- link rotor_3: geometry visual mesh filename=file:///home/hggshiwo/catkin_ws/src/gazebo_sim/models/iris_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 scale=1 1 1
