Commit message: 支持car

File: urdf/catvehicle.xacro (robot description, xacro)
@@ -1,3 +1,3 @@
-<?xml version="1.0" ?>
+<?xml version="1.0"?>
 <!--
 Author: Jonathan Sprinkle, Sam Taylor, Alex Warren, Rahul Bhadani
@@ -29,23 +29,24 @@
 -->
 <robot name="$(arg roboname)" xmlns:xacro="http://www.ros.org/wiki/xacro">
-    <xacro:arg name="updateRate" default="10"/>
-    <xacro:arg name="camera_left" default="true"/>
-    <xacro:arg name="camera_right" default="true"/>
-    <xacro:arg name="triclops" default="true"/>
-    <xacro:arg name="velodyne_points" default="true"/>
-    <xacro:arg name="laser_points" default="true"/>
-    <xacro:property name="velodyne_points" value="$(arg velodyne_points)"/>
-    <xacro:property name="laser_points" value="$(arg laser_points)"/>
-    <xacro:property name="camera_right" value="$(arg camera_right)"/>
-    <xacro:property name="camera_left" value="$(arg camera_left)"/>
-    <xacro:property name="triclops" value="$(arg triclops)"/>
-    <xacro:property name="camera_box" value="0.1"/>
-    <xacro:property name="sensor_box" value="0.25"/>
-    <xacro:property name="PI" value="3.1415926835897931"/>
-    <xacro:property name="base_height" value="1.0639"/>
-    <xacro:property name="base_mass" value="1703.239"/>
-    <!--Car's height is the height of bouding box of the 3D
+    <xacro:arg name="updateRate" default="10" />
+    <xacro:arg name="camera_left" default="true" />
+    <xacro:arg name="camera_right" default="true" />
+    <xacro:arg name="triclops" default="true" />
+    <xacro:arg name="velodyne_points" default="true" />
+    <xacro:arg name="laser_points" default="true" />
+    <xacro:property name="velodyne_points" value="$(arg velodyne_points)" />
+    <xacro:property name="laser_points" value="$(arg laser_points)" />
+    <xacro:property name="camera_right" value="$(arg camera_right)" />
+    <xacro:property name="camera_left" value="$(arg camera_left)" />
+    <xacro:property name="triclops" value="$(arg triclops)" />
+    <xacro:property name="camera_box" value="0.1" />
+    <xacro:property name="sensor_box" value="0.25" />
+    <xacro:property name="PI" value="3.1415926835897931" />
+    <xacro:property name="base_height" value="1.0639" />
+    <xacro:property name="base_mass" value="1703.239" />
+    <!--Car's
+    height is the height of bouding box of the 3D
     mesh given by meshlab -->
-    <xacro:property name="car_height" value="1.5837572084"/>
+    <xacro:property name="car_height" value="1.5837572084" />
     <!-- car_to_bumper is car's length. The value reported here
     is the lenght of the bounding box of the 3D mesh of the car's
@@ -54,32 +55,35 @@
     anywhere -->
     <!-- Wheelbase is roughly 2.8232111 m -->
-    <xacro:property name="car_to_bumper" value="4.4324092962"/>
-    <xacro:property name="car_COM_x" value="-0.0202"/>
-    <xacro:property name="car_COM_y" value="0.0126"/>
-    <xacro:property name="car_COM_z" value="-0.0256"/>
+    <xacro:property name="car_to_bumper" value="4.4324092962" />
+    <xacro:property name="car_COM_x" value="-0.0202" />
+    <xacro:property name="car_COM_y" value="0.0126" />
+    <xacro:property name="car_COM_z" value="-0.0256" />
     <!-- We are assuming that front bumper's height is half of the car's
     bounding box height -->
-    <xacro:property name="front_bumper_height" value="${car_height/2}"/>
-    <!--This is the car tread, i.e distance between right and left front wheels-->
-    <xacro:property name="car_width" value="1.290"/>
-    <xacro:property name="car_width_offset" value="0.05"/>
+    <xacro:property name="front_bumper_height" value="${car_height/2}" />
+    <!--This
+    is the car tread, i.e distance between right and left front wheels-->
+    <xacro:property name="car_width" value="1.290" />
+    <xacro:property name="car_width_offset" value="0.05" />
     <!-- Inertial tensor of car body has been taken from meshlab after
     analyzing the 3D structure of car body -->
-    <xacro:property name="base_mass_ixx" value="347.195805"/>
-    <xacro:property name="base_mass_ixy" value="-11.4914985"/>
-    <xacro:property name="base_mass_ixz" value="18.5070628"/>
-    <xacro:property name="base_mass_iyy" value="2330.10026"/>
-    <xacro:property name="base_mass_iyz" value="3.97814264"/>
-    <xacro:property name="base_mass_izz" value="2529.41827"/>
-    <xacro:property name="tyre_x" value="1.05"/>
-    <xacro:property name="tyre_front_x" value="1.55"/>
-    <xacro:property name="tyre_back_x" value="-1.05"/>
-    <xacro:property name="tyre_y" value="0.765"/>
-    <xacro:property name="tyre_r" value="0.66"/>
-    <!--Below is the thickness of the car's tyre-->
-    <xacro:property name="tyre_length" value="0.2336291492"/>
-    <xacro:property name="tyre_radius" value="0.3671951254"/>
-    <xacro:property name="tyre_mass" value="20"/>
-    <!--xacro:property name="tyre_mass_ixx" value="2.53174430759784"/>
+    <xacro:property name="base_mass_ixx" value="347.195805" />
+    <xacro:property name="base_mass_ixy" value="-11.4914985" />
+    <xacro:property name="base_mass_ixz" value="18.5070628" />
+    <xacro:property name="base_mass_iyy" value="2330.10026" />
+    <xacro:property name="base_mass_iyz" value="3.97814264" />
+    <xacro:property name="base_mass_izz" value="2529.41827" />
+    <xacro:property name="tyre_x" value="1.05" />
+    <xacro:property name="tyre_front_x" value="1.55" />
+    <xacro:property name="tyre_back_x" value="-1.05" />
+    <xacro:property name="tyre_y" value="0.765" />
+    <xacro:property name="tyre_r" value="0.66" />
+    <!--Below
+    is the thickness of the car's tyre-->
+    <xacro:property name="tyre_length" value="0.2336291492" />
+    <xacro:property name="tyre_radius" value="0.3671951254" />
+    <xacro:property name="tyre_mass" value="20" />
+    <!--xacro:property
+    name="tyre_mass_ixx" value="2.53174430759784"/>
     <xacro:property name="tyre_mass_iyy" value="1.43724304615612"/>
     <xacro:property name="tyre_mass_izz" value="1.39917175362076"/>
@@ -90,94 +94,134 @@
     In this model, we didn't use actual mesh of tyre, but a simplified
     cylindrical model. -->
-    <xacro:property name="tyre_mass_ixx" value="${((1/2)*tyre_mass*tyre_radius*tyre_radius)}"/>
-    <xacro:property name="tyre_mass_iyy" value="${((1/12)*tyre_mass*tyre_length*tyre_length) + ((1/4)*tyre_mass*tyre_radius*tyre_radius)}"/>
-    <xacro:property name="tyre_mass_izz" value="${((1/12)*tyre_mass*tyre_length*tyre_length) + ((1/4)*tyre_mass*tyre_radius*tyre_radius)}"/>
-    <xacro:property name="tyre_mass_ixz" value="0.0"/>
-    <xacro:property name="tyre_mass_ixy" value="0.0"/>
-    <xacro:property name="tyre_mass_iyz" value="0.0"/>
-    <xacro:property name="tyre_height" value="-0.696"/>
-    <xacro:property name="str_mass" value="50.00"/>
-    <xacro:property name="str_length" value="0.05"/>
-    <xacro:property name="str_radius" value="0.1"/>
-    <xacro:property name="front_right_offset" value="0.05"/>
-    <xacro:property name="str_mass_ixx" value="${((1/2)*str_mass*str_radius*str_radius)}"/>
-    <xacro:property name="str_mass_iyy" value="${((1/12)*str_mass*str_length*str_length) + ((1/4)*str_mass*str_radius*str_radius)}"/>
-    <xacro:property name="str_mass_izz" value="${((1/12)*str_mass*str_length*str_length) + ((1/4)*str_mass*str_radius*str_radius)}"/>
-    <xacro:property name="str_angle" value="0.6"/>
+    <xacro:property name="tyre_mass_ixx" value="${((1/2)*tyre_mass*tyre_radius*tyre_radius)}" />
+    <xacro:property name="tyre_mass_iyy"
+        value="${((1/12)*tyre_mass*tyre_length*tyre_length) + ((1/4)*tyre_mass*tyre_radius*tyre_radius)}" />
+    <xacro:property name="tyre_mass_izz"
+        value="${((1/12)*tyre_mass*tyre_length*tyre_length) + ((1/4)*tyre_mass*tyre_radius*tyre_radius)}" />
+    <xacro:property name="tyre_mass_ixz" value="0.0" />
+    <xacro:property name="tyre_mass_ixy" value="0.0" />
+    <xacro:property name="tyre_mass_iyz" value="0.0" />
+    <xacro:property name="tyre_height" value="-0.696" />
+    <xacro:property name="str_mass" value="50.00" />
+    <xacro:property name="str_length" value="0.05" />
+    <xacro:property name="str_radius" value="0.1" />
+    <xacro:property name="front_right_offset" value="0.05" />
+    <xacro:property name="str_mass_ixx" value="${((1/2)*str_mass*str_radius*str_radius)}" />
+    <xacro:property name="str_mass_iyy"
+        value="${((1/12)*str_mass*str_length*str_length) + ((1/4)*str_mass*str_radius*str_radius)}" />
+    <xacro:property name="str_mass_izz"
+        value="${((1/12)*str_mass*str_length*str_length) + ((1/4)*str_mass*str_radius*str_radius)}" />
+    <xacro:property name="str_angle" value="0.6" />
     <xacro:property name="tyre_origin">
-        <origin xyz="0 0 0" rpy="${PI/2} 0 0"/>
+        <origin xyz="0 0 0" rpy="${PI/2} 0 0" />
     </xacro:property>
     <xacro:property name="tyre_origin_2">
-        <origin xyz="0 0 0" rpy="0 0 ${PI/2}"/>
+        <origin xyz="0 0 0" rpy="0 0 ${PI/2}" />
     </xacro:property>
     <xacro:property name="tyre_origin_3">
-        <origin xyz="0 0 0" rpy="0 0 ${-PI/2}"/>
+        <origin xyz="0 0 0" rpy="0 0 ${-PI/2}" />
     </xacro:property>
     <xacro:property name="marker_origin">
-        <origin xyz="0 0 0" rpy="0 0 0"/>
+        <origin xyz="0 0 0" rpy="0 0 0" />
     </xacro:property>
-    <xacro:property name="front_laser_size" value="0.25"/>
-    <xacro:property name="front_laser_mass" value="1"/>
-    <xacro:include filename="$(find catvehicle)/urdf/catvehicle.gazebo"/>
+    <xacro:property name="front_laser_size" value="0.25" />
+    <xacro:property name="front_laser_mass" value="1" />
+    <xacro:include filename="$(find catvehicle)/urdf/catvehicle.gazebo" />
     <xacro:if value="${velodyne_points}">
         <!-- You can pass parameters in order to change the max/min
         horizontal angles of the velodyne sensors. These are interpreted
         in the velodyne_points gazebo file -->
-        <xacro:arg name="velodyne_min_angle" default="-0.4"/>
-        <xacro:arg name="velodyne_max_angle" default="0.4"/>
-        <xacro:property name="velodyne_min_angle" value="$(arg velodyne_min_angle)"/>
-        <xacro:property name="velodyne_max_angle" value="$(arg velodyne_max_angle)"/>
-        <xacro:include filename="$(find catvehicle)/urdf/catvehicle_velodyne_points.gazebo"/>
+        <xacro:arg name="velodyne_min_angle" default="-0.4" />
+        <xacro:arg name="velodyne_max_angle" default="0.4" />
+        <xacro:property name="velodyne_min_angle" value="$(arg velodyne_min_angle)" />
+        <xacro:property name="velodyne_max_angle" value="$(arg velodyne_max_angle)" />
+        <xacro:include filename="$(find catvehicle)/urdf/catvehicle_velodyne_points.gazebo" />
     </xacro:if>
     <xacro:if value="${camera_right}">
-        <xacro:include filename="$(find catvehicle)/urdf/catvehicle_right_camera.gazebo"/>
+        <xacro:include filename="$(find catvehicle)/urdf/catvehicle_right_camera.gazebo" />
     </xacro:if>
     <xacro:if value="${camera_left}">
-        <xacro:include filename="$(find catvehicle)/urdf/catvehicle_left_camera.gazebo"/>
+        <xacro:include filename="$(find catvehicle)/urdf/catvehicle_left_camera.gazebo" />
     </xacro:if>
     <xacro:if value="${triclops}">
-        <xacro:include filename="$(find catvehicle)/urdf/catvehicle_triclops.gazebo"/>
+        <xacro:include filename="$(find catvehicle)/urdf/catvehicle_triclops.gazebo" />
     </xacro:if>
     <xacro:if value="${laser_points}">
-        <xacro:include filename="$(find catvehicle)/urdf/catvehicle_laser_points.gazebo"/>
+        <xacro:include filename="$(find catvehicle)/urdf/catvehicle_laser_points.gazebo" />
     </xacro:if>
-    <!--Car Body-->
+    <!--Car
+    Body-->
+    <gazebo>
+        <plugin name="arducopter_plugin" filename="libArduPilotPlugin.so">
+            <fdm_addr>127.0.0.1</fdm_addr>
+            <fdm_port_in>9002</fdm_port_in>
+            <fdm_port_out>9003</fdm_port_out>
+            <!--
+          Require by APM :
+          Only change model and gazebo from XYZ to XY-Z coordinates
+      -->
+            <modelXYZToAirplaneXForwardZDown>0 0 0 3.141593 0 0</modelXYZToAirplaneXForwardZDown>
+            <gazeboXYZToNED>0 0 0 3.141593 0 0</gazeboXYZToNED>
+            <imuName>ugv_0::base_link::imu_sensor</imuName>
+            <connectionTimeoutMaxCount>5</connectionTimeoutMaxCount>
+        </plugin>
+    </gazebo>
+    <gazebo reference="base_link">
+        <sensor name="imu_sensor" type="imu">
+            <always_on>true</always_on>
+            <update_rate>1000</update_rate>
+            <visualize>true</visualize>
+            <topic>__default_topic__</topic>
+            <plugin filename="libgazebo_ros_imu_sensor.so" name="imu_plugin">
+                <topicName>trunk_imu</topicName>
+                <bodyName>base_link</bodyName>
+                <updateRateHZ>1000.0</updateRateHZ>
+                <gaussianNoise>0.0</gaussianNoise>
+                <xyzOffset>0 0 0</xyzOffset>
+                <rpyOffset>0 0 0</rpyOffset>
+                <frameName>base_link</frameName>
+            </plugin>
+            <pose>0 0 0 3.1415926 0 0</pose>
+        </sensor>
+    </gazebo>
     <link name="base_link">
         <collision>
-            <origin xyz="0 0 ${base_height}" rpy="0 0 0"/>
-            <geometry>
-                <mesh filename="package://catvehicle/meshes/ford_escape_no_wheels_2.dae"/>
-            </geometry>
-        </collision>
-        <visual>
-            <origin xyz="0 0 ${base_height}" rpy="0 0 0"/>
-            <geometry>
-                <mesh filename="package://catvehicle/meshes/ford_escape_no_wheels_2.dae"/>
+            <origin xyz="0 0 ${base_height}" rpy="0 0 0" />
+            <geometry>
+                <mesh filename="package://catvehicle/meshes/ford_escape_no_wheels_2.dae" />
+            </geometry>
+        </collision>
+        <visual>
+            <origin xyz="0 0 ${base_height}" rpy="0 0 0" />
+            <geometry>
+                <mesh filename="package://catvehicle/meshes/ford_escape_no_wheels_2.dae" />
             </geometry>
         </visual>
     </link>
     <joint name="inertial_joint" type="fixed">
-        <parent link="base_link"/>
-        <child link="main_mass"/>
-        <origin xyz="0 0 0" rpy="0 0 0"/>
+        <parent link="base_link" />
+        <child link="main_mass" />
+        <origin xyz="0 0 0" rpy="0 0 0" />
     </joint>
     <link name="main_mass" type="fixed">
-        <parent link="inertial_joint"/>
-        <inertial>
-            <origin xyz="${car_COM_x} ${car_COM_y} ${car_COM_z}" rpy="0 0 0"/> <!-- This is the center of mass of Car Body-->
-            <mass value="${base_mass}"/>
+        <parent link="inertial_joint" />
+        <inertial>
+            <origin xyz="${car_COM_x} ${car_COM_y} ${car_COM_z}" rpy="0 0 0" /> <!-- This is the
+            center of mass of Car Body-->
+            <mass value="${base_mass}" />
             <inertia
-            ixx="${base_mass_ixx}"  ixy="${base_mass_ixy}" ixz="${base_mass_ixz}"
-            iyy="${base_mass_iyy}" iyz="${base_mass_iyz}"
-            izz="${base_mass_izz}"/>
-        </inertial>
-    </link>
-    <!--Back Right Wheel-->
+                ixx="${base_mass_ixx}" ixy="${base_mass_ixy}" ixz="${base_mass_ixz}"
+                iyy="${base_mass_iyy}" iyz="${base_mass_iyz}"
+                izz="${base_mass_izz}" />
+        </inertial>
+    </link>
+    <!--Back
+    Right Wheel-->
     <joint name="back_right_wheel_joint" type="continuous">
-        <parent link="base_link"/>
-        <child link="back_right_wheel_link"/>
-        <origin xyz="${tyre_back_x} ${-tyre_y} ${tyre_r}" rpy="0 0 0"/>
-        <axis xyz="0 1 0"/>
-        <dynamics damping="0.01"/>
+        <parent link="base_link" />
+        <child link="back_right_wheel_link" />
+        <origin xyz="${tyre_back_x} ${-tyre_y} ${tyre_r}" rpy="0 0 0" />
+        <axis xyz="0 1 0" />
+        <dynamics damping="0.01" />
         <limit effort="10000" velocity="1000" />
         <joint_properties damping="10" friction="10.0" />
@@ -185,8 +229,9 @@
     <link name="back_right_wheel_link">
         <collision>
-            <origin xyz="0 0 0" rpy="${PI/2} 0 0"/>
-            <geometry>
-                <cylinder length="${tyre_length}" radius="${tyre_radius}"/>
-                <!--mesh filename="package://catvehicle/meshes/ford_escape_wheel.dae"/-->
+            <origin xyz="0 0 0" rpy="${PI/2} 0 0" />
+            <geometry>
+                <cylinder length="${tyre_length}" radius="${tyre_radius}" />
+                <!--mesh
+                filename="package://catvehicle/meshes/ford_escape_wheel.dae"/-->
             </geometry>
             <surface>
@@ -211,28 +256,31 @@
         </collision>
         <visual>
-            <!--origin xyz="0 0 0" rpy="${PI/2} 0 0"/-->
-            <origin xyz="0 ${car_width_offset*2} 0.0" rpy="0 0 ${-PI/2}"/>
-            <geometry>
-                <!--cylinder length="${tyre_length}" radius="${tyre_radius}"/>
+            <!--origin
+            xyz="0 0 0" rpy="${PI/2} 0 0"/-->
+            <origin xyz="0 ${car_width_offset*2} 0.0" rpy="0 0 ${-PI/2}" />
+            <geometry>
+                <!--cylinder
+                length="${tyre_length}" radius="${tyre_radius}"/>
                 <scale xyz="1 1 1"/-->
-                <mesh scale="1.2 1 1" filename="package://catvehicle/meshes/ford_escape_wheel.dae"/>
-            </geometry>
-        </visual>
-        <inertial>
-            <origin xyz="0 0 0" rpy="0 0 0"/>
-            <mass value="${tyre_mass}"/>
+                <mesh scale="1.2 1 1" filename="package://catvehicle/meshes/ford_escape_wheel.dae" />
+            </geometry>
+        </visual>
+        <inertial>
+            <origin xyz="0 0 0" rpy="0 0 0" />
+            <mass value="${tyre_mass}" />
             <inertia
-            ixx="${tyre_mass_ixx}"  ixy="${tyre_mass_ixy}"  ixz="${tyre_mass_ixz}"
-            iyy="${tyre_mass_iyy}"  iyz="${tyre_mass_iyz}"
-            izz="${tyre_mass_izz}"/>
-        </inertial>
-    </link>
-    <!--Back Left Wheel -->
+                ixx="${tyre_mass_ixx}" ixy="${tyre_mass_ixy}" ixz="${tyre_mass_ixz}"
+                iyy="${tyre_mass_iyy}" iyz="${tyre_mass_iyz}"
+                izz="${tyre_mass_izz}" />
+        </inertial>
+    </link>
+    <!--Back
+    Left Wheel -->
     <joint name="back_left_wheel_joint" type="continuous">
-        <parent link="base_link"/>
-        <child link="back_left_wheel_link"/>
-        <origin xyz="${tyre_back_x} ${tyre_y} ${tyre_r}" rpy="0 0 0"/>
-        <axis xyz="0 1 0"/>
-        <dynamics damping="0.01"/>
+        <parent link="base_link" />
+        <child link="back_left_wheel_link" />
+        <origin xyz="${tyre_back_x} ${tyre_y} ${tyre_r}" rpy="0 0 0" />
+        <axis xyz="0 1 0" />
+        <dynamics damping="0.01" />
         <limit effort="10000" velocity="1000" />
         <joint_properties damping="10" friction="10.0" />
@@ -240,8 +288,9 @@
     <link name="back_left_wheel_link">
         <collision>
-            <origin xyz="0 0 0" rpy="${PI/2} 0 0"/>
-            <geometry>
-                <cylinder length="${tyre_length}" radius="${tyre_radius}"/>
-                <!--mesh filename="package://catvehicle/meshes/ford_escape_wheel.dae"/-->
+            <origin xyz="0 0 0" rpy="${PI/2} 0 0" />
+            <geometry>
+                <cylinder length="${tyre_length}" radius="${tyre_radius}" />
+                <!--mesh
+                filename="package://catvehicle/meshes/ford_escape_wheel.dae"/-->
             </geometry>
             <surface>
@@ -266,67 +315,73 @@
         </collision>
         <visual>
-            <!--origin xyz="0 0 0" rpy="${PI/2} 0 0"/-->
-            <origin xyz="0 ${-car_width_offset*2} 0.0" rpy="0 0 ${PI/2}"/>
-            <geometry>
-                <!--cylinder length="${tyre_length}" radius="${tyre_radius}"/-->
-                <mesh scale="1.2 1 1" filename="package://catvehicle/meshes/ford_escape_wheel.dae"/>
-            </geometry>
-        </visual>
-        <inertial>
-            <origin xyz="0 0 0" rpy="0 0 0"/>
-            <mass value="${tyre_mass}"/>
+            <!--origin
+            xyz="0 0 0" rpy="${PI/2} 0 0"/-->
+            <origin xyz="0 ${-car_width_offset*2} 0.0" rpy="0 0 ${PI/2}" />
+            <geometry>
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